File: hardware/keyboard2018.sch (KiCad schematic (older format))
At the start: 7 parts, among them J1 USB_B_Micro, U1 PIC16F1454-IP, U2 PIC16F18854-IP

Commit message: Switch (haha) from F18854 to F18855
Parts:
- removed U2: PIC16F18854-IP, Package_DIP:DIP-28_W7.62mm_Socket, symbol custom-pic:PIC16F18854-IP
- added U2: PIC16F18855-IP, symbol custom-pic:PIC16F18855-IP
Changed lines of the file:
@@
 Wire Wire Line
 	4650 4250 4550 4250
-$Comp
-L custom-pic:PIC16F18854-IP U2
-U 1 1 5B8FD9EB
-P 6750 4050
-F 0 "U2" V 6771 2922 50  0000 R CNN
-F 1 "PIC16F18854-IP" V 6680 2922 50  0000 R CNN
-F 2 "Package_DIP:DIP-28_W7.62mm_Socket" H 6700 5250 50  0001 C CNN
-F 3 "" H 6700 5250 50  0001 C CNN
-	1    6750 4050
-	0    -1   -1   0
-$EndComp
 Wire Wire Line
 	800  4250 1250 4250
@@
 NoConn ~ 1550 1650
 Wire Bus Line
+	7400 5200 8700 5200
+Wire Bus Line
+	4750 2950 8700 2950
+Wire Bus Line
 	5600 5200 7250 5200
 Wire Bus Line
@@
 Wire Bus Line
 	4050 4950 4050 6350
-Wire Bus Line
-	4750 2950 8700 2950
-Wire Bus Line
-	7400 5200 8700 5200
+$Comp
+L custom-pic:PIC16F18855-IP U2
+U 1 1 5B8F2463
+P 6750 4050
+F 0 "U2" V 6771 2922 50  0000 R CNN
+F 1 "PIC16F18855-IP" V 6680 2922 50  0000 R CNN
+F 2 "" H 6700 5250 50  0001 C CNN
+F 3 "" H 6700 5250 50  0001 C CNN
+	1    6750 4050
+	0    -1   -1   0
+$EndComp
 $EndSCHEMATC

Commit message: Finish schematic
Parts:
- added J2: Conn_01x05_Male, symbol Connector:Conn_01x05_Male
Changed lines of the file:
@@
 L power:GND #PWR0103
 U 1 1 5C596273
-P 3750 1450
-F 0 "#PWR0103" H 3750 1200 50  0001 C CNN
-F 1 "GND" H 3755 1277 50  0000 C CNN
-F 2 "" H 3750 1450 50  0001 C CNN
-F 3 "" H 3750 1450 50  0001 C CNN
-	1    3750 1450
+P 3450 1400
+F 0 "#PWR0103" H 3450 1150 50  0001 C CNN
+F 1 "GND" H 3455 1227 50  0000 C CNN
+F 2 "" H 3450 1400 50  0001 C CNN
+F 3 "" H 3450 1400 50  0001 C CNN
+	1    3450 1400
 	1    0    0    -1
 $EndComp
@@
 	3850 3800 3750 3800
 Wire Wire Line
-	3600 1450 3750 1450
+	3300 1400 3450 1400
 Text Label 3800 4400 0    50   ~ 0
 ICSPDAT_EXT
@@
 Wire Wire Line
 	1900 3800 1950 3800
-Text Label 3650 1050 0    50   ~ 0
+Text Label 3350 1200 0    50   ~ 0
 ICSPDAT_EXT
-Text Label 3650 1350 0    50   ~ 0
+Text Label 3350 1300 0    50   ~ 0
 ICSPCLK_EXT
-Text Label 3650 950  0    50   ~ 0
+Text Label 3350 1100 0    50   ~ 0
 ~MCLR~_EXT
 Wire Wire Line
@@
 NoConn ~ 6550 3450
 Wire Wire Line
-	3600 1350 4150 1350
-Wire Wire Line
-	3600 1050 4150 1050
-Wire Wire Line
-	3600 950  4150 950
-Wire Wire Line
-	3600 1150 4050 1150
+	3300 1300 3850 1300
+Wire Wire Line
+	3300 1200 3850 1200
+Wire Wire Line
+	3300 1100 3850 1100
+Wire Wire Line
+	3300 1000 3750 1000
 $Comp
 L power:VDD #PWR0107
 U 1 1 5C36F0D2
-P 4050 1150
-F 0 "#PWR0107" H 4050 1000 50  0001 C CNN
-F 1 "VDD" V 4067 1278 50  0000 L CNN
-F 2 "" H 4050 1150 50  0001 C CNN
-F 3 "" H 4050 1150 50  0001 C CNN
-	1    4050 1150
+P 3750 1000
+F 0 "#PWR0107" H 3750 850 50  0001 C CNN
+F 1 "VDD" V 3767 1128 50  0000 L CNN
+F 2 "" H 3750 1000 50  0001 C CNN
+F 3 "" H 3750 1000 50  0001 C CNN
+	1    3750 1000
 	0    1    1    0
 $EndComp
 NoConn ~ 1550 1650
-Wire Bus Line
-	7400 5200 8700 5200
-Wire Bus Line
-	4750 2950 8700 2950
-Wire Bus Line
-	5600 5200 7250 5200
-Wire Bus Line
-	5600 5200 5600 6350
-Wire Bus Line
-	4050 4950 4050 6350
 $Comp
 L custom-pic:PIC16F18855-IP U2
@@
 	0    -1   -1   0
 $EndComp
+Wire Bus Line
+	7400 5200 8700 5200
+Wire Bus Line
+	4750 2950 8700 2950
+Wire Bus Line
+	5600 5200 7250 5200
+Wire Bus Line
+	5600 5200 5600 6350
+Wire Bus Line
+	4050 4950 4050 6350
+$Comp
+L Connector:Conn_01x05_Male J2
+U 1 1 5B97994E
+P 3100 1200
+F 0 "J2" H 3200 1550 50  0000 C CNN
+F 1 "Conn_01x05_Male" H 3206 1487 50  0001 C CNN
+F 2 "" H 3100 1200 50  0001 C CNN
+F 3 "~" H 3100 1200 50  0001 C CNN
+	1    3100 1200
+	1    0    0    -1
+$EndComp
 $EndSCHEMATC

Commit message: Assign a couple more footprints
Parts:
- J2: footprint (none) -> Connector_PinHeader_2.54mm:PinHeader_1x05_P2.54mm_Horizontal
- U2: footprint (none) -> Package_DIP:DIP-28_W7.62mm_Socket
Changed lines of the file:
@@
 F 0 "U2" V 6771 2922 50  0000 R CNN
 F 1 "PIC16F18855-IP" V 6680 2922 50  0000 R CNN
-F 2 "" H 6700 5250 50  0001 C CNN
+F 2 "Package_DIP:DIP-28_W7.62mm_Socket" H 6700 5250 50  0001 C CNN
 F 3 "" H 6700 5250 50  0001 C CNN
 	1    6750 4050
@@
 F 0 "J2" H 3200 1550 50  0000 C CNN
 F 1 "Conn_01x05_Male" H 3206 1487 50  0001 C CNN
-F 2 "" H 3100 1200 50  0001 C CNN
+F 2 "Connector_PinHeader_2.54mm:PinHeader_1x05_P2.54mm_Horizontal" H 3100 1200 50  0001 C CNN
 F 3 "~" H 3100 1200 50  0001 C CNN
 	1    3100 1200

Commit message: Finish schematic again
Parts:
- added SW1: SW_Push, custom:TE FSM4JAH, symbol Switch:SW_Push
Connections:
- wire segments 78 -> 79
Changed lines of the file:
@@
 	0    -1   -1   0
+$EndComp
+$Comp
+L Connector:Conn_01x05_Male J2
+U 1 1 5B97994E
+P 3100 1200
+F 0 "J2" H 3200 1550 50  0000 C CNN
+F 1 "Conn_01x05_Male" H 3206 1487 50  0001 C CNN
+F 2 "Connector_PinHeader_2.54mm:PinHeader_1x05_P2.54mm_Horizontal" H 3100 1200 50  0001 C CNN
+F 3 "~" H 3100 1200 50  0001 C CNN
+	1    3100 1200
+	1    0    0    -1
+$EndComp
+Wire Wire Line
+	1250 4250 1250 4800
+$Comp
+L Switch:SW_Push SW1
+U 1 1 5B95ED3D
+P 1250 5000
+F 0 "SW1" V 1250 5148 50  0000 L CNN
+F 1 "SW_Push" V 1295 5148 50  0001 L CNN
+F 2 "custom:TE FSM4JAH" H 1250 5200 50  0001 C CNN
+F 3 "" H 1250 5200 50  0001 C CNN
+	1    1250 5000
+	0    1    1    0
+$EndComp
+$Comp
+L power:GND #PWR0109
+U 1 1 5B979F84
+P 1250 5200
+F 0 "#PWR0109" H 1250 4950 50  0001 C CNN
+F 1 "GND" H 1255 5027 50  0000 C CNN
+F 2 "" H 1250 5200 50  0001 C CNN
+F 3 "" H 1250 5200 50  0001 C CNN
+	1    1250 5200
+	1    0    0    -1
 $EndComp
 Wire Bus Line
@@
 Wire Bus Line
 	4050 4950 4050 6350
-$Comp
-L Connector:Conn_01x05_Male J2
-U 1 1 5B97994E
-P 3100 1200
-F 0 "J2" H 3200 1550 50  0000 C CNN
-F 1 "Conn_01x05_Male" H 3206 1487 50  0001 C CNN
-F 2 "Connector_PinHeader_2.54mm:PinHeader_1x05_P2.54mm_Horizontal" H 3100 1200 50  0001 C CNN
-F 3 "~" H 3100 1200 50  0001 C CNN
-	1    3100 1200
-	1    0    0    -1
-$EndComp
 $EndSCHEMATC

Commit message: Switch USB connector
Parts:
- removed J1: USB_B_Micro, Connector_USB:USB_Mini-B_Lumberg_2486_01_Horizontal, symbol Connector:USB_B_Micro
- added J1: USB_B, custom:captive USB, symbol Connector:USB_B
Connections:
- no-connect marks 5 -> 4
Changed lines of the file:
@@
 $EndDescr
-$Comp
-L Connector:USB_B_Micro J1
-U 1 1 5B8779DB
-P 1650 1250
-F 0 "J1" H 1705 1717 50  0000 C CNN
-F 1 "USB_B_Micro" H 1705 1626 50  0000 C CNN
-F 2 "Connector_USB:USB_Mini-B_Lumberg_2486_01_Horizontal" H 1800 1200 50  0001 C CNN
-F 3 "~" H 1800 1200 50  0001 C CNN
-	1    1650 1250
-	1    0    0    -1
-$EndComp
 $Comp
 L power:GND #PWR0101
 U 1 1 5B879A94
-P 1650 1700
-F 0 "#PWR0101" H 1650 1450 50  0001 C CNN
-F 1 "GND" H 1655 1527 50  0000 C CNN
-F 2 "" H 1650 1700 50  0001 C CNN
-F 3 "" H 1650 1700 50  0001 C CNN
-	1    1650 1700
-	1    0    0    -1
-$EndComp
-Wire Wire Line
-	1650 1700 1650 1650
+P 1400 1700
+F 0 "#PWR0101" H 1400 1450 50  0001 C CNN
+F 1 "GND" H 1405 1527 50  0000 C CNN
+F 2 "" H 1400 1700 50  0001 C CNN
+F 3 "" H 1400 1700 50  0001 C CNN
+	1    1400 1700
+	1    0    0    -1
+$EndComp
+Wire Wire Line
+	1400 1700 1400 1650
 $Comp
 L power:GND #PWR0102
@@
 	1    0    0    -1
 $EndComp
-NoConn ~ 1950 1450
 $Comp
 L power:GND #PWR0120
@@
 D-
 Wire Wire Line
-	2150 1250 1950 1250
-Wire Wire Line
-	2150 1350 1950 1350
-Text Label 2000 1350 0    50   ~ 0
+	1900 1250 1700 1250
+Wire Wire Line
+	1900 1350 1700 1350
+Text Label 1750 1350 0    50   ~ 0
 D-
-Text Label 2000 1250 0    50   ~ 0
+Text Label 1750 1250 0    50   ~ 0
 D+
 $Comp
 L power:VDD #PWR0127
 U 1 1 5B8F9546
-P 2050 1050
-F 0 "#PWR0127" H 2050 900 50  0001 C CNN
-F 1 "VDD" V 2067 1178 50  0000 L CNN
-F 2 "" H 2050 1050 50  0001 C CNN
-F 3 "" H 2050 1050 50  0001 C CNN
-	1    2050 1050
+P 1800 1050
+F 0 "#PWR0127" H 1800 900 50  0001 C CNN
+F 1 "VDD" V 1817 1178 50  0000 L CNN
+F 2 "" H 1800 1050 50  0001 C CNN
+F 3 "" H 1800 1050 50  0001 C CNN
+	1    1800 1050
 	0    1    1    0
 $EndComp
 Wire Wire Line
-	2050 1050 1950 1050
+	1800 1050 1700 1050
 Wire Wire Line
 	4650 4250 4550 4250
@@
 	0    1    1    0
 $EndComp
-NoConn ~ 1550 1650
 $Comp
 L custom-pic:PIC16F18855-IP U2
@@
 	1    0    0    -1
 $EndComp
+$Comp
+L Connector:USB_B J1
+U 1 1 5B9AB7F1
+P 1400 1250
+F 0 "J1" H 1455 1717 50  0000 C CNN
+F 1 "USB_B" H 1455 1626 50  0000 C CNN
+F 2 "custom:captive USB" H 1550 1200 50  0001 C CNN
+F 3 " ~" H 1550 1200 50  0001 C CNN
+	1    1400 1250
+	1    0    0    -1
+$EndComp
+NoConn ~ 1300 1650
 Wire Bus Line
 	7400 5200 8700 5200

Commit message: Decent layout
Parts:
- added TP1, TP2, TP3: TestPoint, custom:test point 1mm, symbol Connector:TestPoint
Connections:
- wire segments 79 -> 80
Changed lines of the file:
@@
 L Device:C C2
 U 1 1 5B87A5A4
-P 4400 4250
-F 0 "C2" V 4148 4250 50  0000 C CNN
-F 1 "470n" V 4239 4250 50  0000 C CNN
-F 2 "Capacitor_THT:C_Disc_D3.0mm_W1.6mm_P2.50mm" H 4438 4100 50  0001 C CNN
-F 3 "~" H 4400 4250 50  0001 C CNN
-	1    4400 4250
+P 4450 4250
+F 0 "C2" V 4198 4250 50  0000 C CNN
+F 1 "470n" V 4289 4250 50  0000 C CNN
+F 2 "Capacitor_THT:C_Disc_D3.0mm_W1.6mm_P2.50mm" H 4488 4100 50  0001 C CNN
+F 3 "~" H 4450 4250 50  0001 C CNN
+	1    4450 4250
 	0    1    1    0
 $EndComp
@@
 L power:GND #PWR0120
 U 1 1 5C5A6BA2
-P 4650 4250
-F 0 "#PWR0120" H 4650 4000 50  0001 C CNN
-F 1 "GND" V 4655 4122 50  0000 R CNN
-F 2 "" H 4650 4250 50  0001 C CNN
-F 3 "" H 4650 4250 50  0001 C CNN
-	1    4650 4250
+P 4700 4250
+F 0 "#PWR0120" H 4700 4000 50  0001 C CNN
+F 1 "GND" V 4705 4122 50  0000 R CNN
+F 2 "" H 4700 4250 50  0001 C CNN
+F 3 "" H 4700 4250 50  0001 C CNN
+	1    4700 4250
 	0    -1   -1   0
 $EndComp
@@
 Connection ~ 1250 4250
 Wire Wire Line
-	3750 4250 4250 4250
-Wire Wire Line
 	3950 3950 3750 3950
 Wire Wire Line
@@
 	1800 1050 1700 1050
 Wire Wire Line
-	4650 4250 4550 4250
+	4700 4250 4600 4250
 Wire Wire Line
 	800  4250 1250 4250
@@
 $EndComp
 NoConn ~ 1300 1650
+$Comp
+L Connector:TestPoint TP1
+U 1 1 5B9C521E
+P 5300 1250
+F 0 "TP1" V 5300 1437 50  0000 L CNN
+F 1 "TestPoint" H 5300 1484 50  0001 C CNN
+F 2 "custom:test point 1mm" H 5500 1250 50  0001 C CNN
+F 3 "~" H 5500 1250 50  0001 C CNN
+	1    5300 1250
+	0    1    1    0
+$EndComp
+$Comp
+L Connector:TestPoint TP2
+U 1 1 5B9C593E
+P 5300 1100
+F 0 "TP2" V 5300 1287 50  0000 L CNN
+F 1 "TestPoint" H 5358 1129 50  0001 L CNN
+F 2 "custom:test point 1mm" H 5500 1100 50  0001 C CNN
+F 3 "~" H 5500 1100 50  0001 C CNN
+	1    5300 1100
+	0    1    1    0
+$EndComp
+$Comp
+L power:GND #PWR0111
+U 1 1 5B9C6172
+P 5300 1250
+F 0 "#PWR0111" H 5300 1000 50  0001 C CNN
+F 1 "GND" V 5305 1122 50  0000 R CNN
+F 2 "" H 5300 1250 50  0001 C CNN
+F 3 "" H 5300 1250 50  0001 C CNN
+	1    5300 1250
+	0    1    1    0
+$EndComp
+$Comp
+L power:VDD #PWR0113
+U 1 1 5B9C61BC
+P 5300 1100
+F 0 "#PWR0113" H 5300 950 50  0001 C CNN
+F 1 "VDD" V 5318 1227 50  0000 L CNN
+F 2 "" H 5300 1100 50  0001 C CNN
+F 3 "" H 5300 1100 50  0001 C CNN
+	1    5300 1100
+	0    -1   -1   0
+$EndComp
+$Comp
+L Connector:TestPoint TP3
+U 1 1 5B9EF05B
+P 4200 4250
+F 0 "TP3" H 4200 4484 50  0000 C CNN
+F 1 "TestPoint" H 4258 4279 50  0001 L CNN
+F 2 "custom:test point 1mm" H 4400 4250 50  0001 C CNN
+F 3 "~" H 4400 4250 50  0001 C CNN
+	1    4200 4250
+	1    0    0    -1
+$EndComp
+Connection ~ 4200 4250
+Wire Wire Line
+	4200 4250 4300 4250
+Wire Wire Line
+	3750 4250 4200 4250
 Wire Bus Line
 	7400 5200 8700 5200

Commit message: checkpoint reached
Parts:
- removed J1: USB_B, custom:captive USB, symbol Connector:USB_B
- added J1: USB_B_no_shield, custom:captive USB, symbol custom:USB_B_no_shield
- U1: symbol custom-pic:PIC16F1454-IP -> custom:PIC16F1454-IP
- U2: symbol custom-pic:PIC16F18855-IP -> custom:PIC16F18855-IP
Connections:
- wire segments 80 -> 83
- no-connect marks 4 -> 0
Changed lines of the file:
@@
 Comment4 ""
 $EndDescr
-$Comp
-L power:GND #PWR0101
-U 1 1 5B879A94
-P 1400 1700
-F 0 "#PWR0101" H 1400 1450 50  0001 C CNN
-F 1 "GND" H 1405 1527 50  0000 C CNN
-F 2 "" H 1400 1700 50  0001 C CNN
-F 3 "" H 1400 1700 50  0001 C CNN
-	1    1400 1700
-	1    0    0    -1
-$EndComp
 Wire Wire Line
 	1400 1700 1400 1650
@@
 Text Label 1500 4700 0    50   ~ 0
 ICSPDAT_INT
-NoConn ~ 2000 3950
-$Comp
-L custom-pic:PIC16F1454-IP U1
+$Comp
+L custom:PIC16F1454-IP U1
 U 1 1 5B8FD686
 P 2850 4250
@@
 Text Label 4400 4950 0    50   ~ 0
 ROW[1..10]
-NoConn ~ 6400 3450
-NoConn ~ 6550 3450
 Wire Wire Line
 	3300 1300 3850 1300
@@
 $EndComp
 $Comp
-L custom-pic:PIC16F18855-IP U2
+L custom:PIC16F18855-IP U2
 U 1 1 5B8F2463
 P 6750 4050
@@
 	1    0    0    -1
 $EndComp
-$Comp
-L Connector:USB_B J1
-U 1 1 5B9AB7F1
-P 1400 1250
-F 0 "J1" H 1455 1717 50  0000 C CNN
-F 1 "USB_B" H 1455 1626 50  0000 C CNN
-F 2 "custom:captive USB" H 1550 1200 50  0001 C CNN
-F 3 " ~" H 1550 1200 50  0001 C CNN
-	1    1400 1250
-	1    0    0    -1
-$EndComp
-NoConn ~ 1300 1650
 $Comp
 L Connector:TestPoint TP1
@@
 Wire Wire Line
 	3750 4250 4200 4250
+$Comp
+L power:GND #PWR0115
+U 1 1 5B976D7D
+P 6400 3400
+F 0 "#PWR0115" H 6400 3150 50  0001 C CNN
+F 1 "GND" H 6405 3227 50  0000 C CNN
+F 2 "" H 6400 3400 50  0001 C CNN
+F 3 "" H 6400 3400 50  0001 C CNN
+	1    6400 3400
+	-1   0    0    1
+$EndComp
+$Comp
+L power:GND #PWR0117
+U 1 1 5B976DDB
+P 6550 3400
+F 0 "#PWR0117" H 6550 3150 50  0001 C CNN
+F 1 "GND" H 6555 3227 50  0000 C CNN
+F 2 "" H 6550 3400 50  0001 C CNN
+F 3 "" H 6550 3400 50  0001 C CNN
+	1    6550 3400
+	-1   0    0    1
+$EndComp
+Wire Wire Line
+	6550 3400 6550 3450
+Wire Wire Line
+	6400 3400 6400 3450
+$Comp
+L power:GND #PWR0129
+U 1 1 5B9810E8
+P 1950 3950
+F 0 "#PWR0129" H 1950 3700 50  0001 C CNN
+F 1 "GND" V 1955 3822 50  0000 R CNN
+F 2 "" H 1950 3950 50  0001 C CNN
+F 3 "" H 1950 3950 50  0001 C CNN
+	1    1950 3950
+	0    1    1    0
+$EndComp
+Wire Wire Line
+	1950 3950 2000 3950
+$Comp
+L custom:USB_B_no_shield J1
+U 1 1 5B99B6A0
+P 1450 1250
+F 0 "J1" H 1455 1717 50  0000 C CNN
+F 1 "USB_B_no_shield" H 1455 1626 50  0000 C CNN
+F 2 "custom:captive USB" H 1400 1700 50  0001 C CNN
+F 3 "" H 1400 1700 50  0001 C CNN
+	1    1450 1250
+	1    0    0    -1
+$EndComp
+$Comp
+L power:GND #PWR0101
+U 1 1 5B99BB93
+P 1400 1700
+F 0 "#PWR0101" H 1400 1450 50  0001 C CNN
+F 1 "GND" H 1405 1527 50  0000 C CNN
+F 2 "" H 1400 1700 50  0001 C CNN
+F 3 "" H 1400 1700 50  0001 C CNN
+	1    1400 1700
+	1    0    0    -1
+$EndComp
 Wire Bus Line
 	7400 5200 8700 5200
