File: hardware/keyboard2018.kicad_pcb (KiCad board)
At the start: 2 copper layers, 0 parts

Commit message: Decent layout
Parts:
- added C1: 100n, Capacitor_THT:C_Disc_D3.0mm_W1.6mm_P2.50mm, B.Cu at (195.6, 138.4)
- added C2: 470n, Capacitor_THT:C_Disc_D3.0mm_W1.6mm_P2.50mm, B.Cu at (188.0, 138.4)
- added C3: 100n, Capacitor_THT:C_Disc_D3.0mm_W1.6mm_P2.50mm, B.Cu at (264.8, 161.9)
- added D_A1: D, Diode_THT:D_A-405_P7.62mm_Horizontal, B.Cu at (80.0, 219.1)
- added D_A10: D, Diode_THT:D_A-405_P7.62mm_Horizontal, B.Cu at (257.8, 219.1)
- added D_A11: D, Diode_THT:D_A-405_P7.62mm_Horizontal, B.Cu at (283.2, 219.1)
- added D_A12: D, Diode_THT:D_A-405_P7.62mm_Horizontal, B.Cu at (302.3, 219.1)
- added D_A13: D, Diode_THT:D_A-405_P7.62mm_Horizontal, B.Cu at (321.3, 219.1)
- added D_A14: D, Diode_THT:D_A-405_P7.62mm_Horizontal, B.Cu at (340.4, 219.1)
- added D_A15: D, Diode_THT:D_A-405_P7.62mm_Horizontal, B.Cu at (359.4, 219.1)
- added D_A16: D, Diode_THT:D_A-405_P7.62mm_Horizontal, B.Cu at (378.5, 219.1)
- added D_A2: D, Diode_THT:D_A-405_P7.62mm_Horizontal, B.Cu at (99.1, 219.1)
- added D_A3: D, Diode_THT:D_A-405_P7.62mm_Horizontal, B.Cu at (118.1, 219.1)
- added D_A4: D, Diode_THT:D_A-405_P7.62mm_Horizontal, B.Cu at (137.2, 219.1)
- added D_A5: D, Diode_THT:D_A-405_P7.62mm_Horizontal, B.Cu at (156.2, 219.1)
- added D_A6: D, Diode_THT:D_A-405_P7.62mm_Horizontal, B.Cu at (175.3, 219.1)
- added D_A7: D, Diode_THT:D_A-405_P7.62mm_Horizontal, B.Cu at (200.7, 219.1)
- added D_A8: D, Diode_THT:D_A-405_P7.62mm_Horizontal, B.Cu at (219.7, 219.1)
- added D_A9: D, Diode_THT:D_A-405_P7.62mm_Horizontal, B.Cu at (238.8, 219.1)
- added D_B1: D, Diode_THT:D_A-405_P7.62mm_Horizontal, B.Cu at (80.0, 200.0)
- added D_B10: D, Diode_THT:D_A-405_P7.62mm_Horizontal, B.Cu at (257.8, 200.0)
- added D_B11: D, Diode_THT:D_A-405_P7.62mm_Horizontal, B.Cu at (283.2, 200.0)
- added D_B12: D, Diode_THT:D_A-405_P7.62mm_Horizontal, B.Cu at (302.3, 200.0)
- added D_B13: D, Diode_THT:D_A-405_P7.62mm_Horizontal, B.Cu at (321.3, 200.0)
- added D_B14: D, Diode_THT:D_A-405_P7.62mm_Horizontal, B.Cu at (340.4, 200.0)
- added D_B15: D, Diode_THT:D_A-405_P7.62mm_Horizontal, B.Cu at (359.4, 200.0)
- added D_B16: D, Diode_THT:D_A-405_P7.62mm_Horizontal, B.Cu at (378.5, 200.0)
- added D_B2: D, Diode_THT:D_A-405_P7.62mm_Horizontal, B.Cu at (99.1, 200.0)
- added D_B3: D, Diode_THT:D_A-405_P7.62mm_Horizontal, B.Cu at (118.1, 200.0)
- added D_B4: D, Diode_THT:D_A-405_P7.62mm_Horizontal, B.Cu at (137.2, 200.0)
- added D_B5: D, Diode_THT:D_A-405_P7.62mm_Horizontal, B.Cu at (156.2, 200.0)
- added D_B6: D, Diode_THT:D_A-405_P7.62mm_Horizontal, B.Cu at (175.3, 200.0)
- added D_B7: D, Diode_THT:D_A-405_P7.62mm_Horizontal, B.Cu at (200.7, 200.0)
- added D_B8: D, Diode_THT:D_A-405_P7.62mm_Horizontal, B.Cu at (219.7, 200.0)
- added D_B9: D, Diode_THT:D_A-405_P7.62mm_Horizontal, B.Cu at (238.8, 200.0)
- added D_C1: D, Diode_THT:D_A-405_P7.62mm_Horizontal, B.Cu at (80.0, 181.0)
- added D_C10: D, Diode_THT:D_A-405_P7.62mm_Horizontal, B.Cu at (257.8, 181.0)
- added D_C11: D, Diode_THT:D_A-405_P7.62mm_Horizontal, B.Cu at (283.2, 181.0)
- added D_C12: D, Diode_THT:D_A-405_P7.62mm_Horizontal, B.Cu at (302.3, 181.0)
- added D_C13: D, Diode_THT:D_A-405_P7.62mm_Horizontal, B.Cu at (321.3, 181.0)
- added D_C14: D, Diode_THT:D_A-405_P7.62mm_Horizontal, B.Cu at (340.4, 181.0)
- added D_C15: D, Diode_THT:D_A-405_P7.62mm_Horizontal, B.Cu at (359.4, 181.0)
- added D_C16: D, Diode_THT:D_A-405_P7.62mm_Horizontal, B.Cu at (378.5, 181.0)
- added D_C2: D, Diode_THT:D_A-405_P7.62mm_Horizontal, B.Cu at (99.1, 181.0)
- added D_C3: D, Diode_THT:D_A-405_P7.62mm_Horizontal, B.Cu at (118.1, 181.0)
- added D_C4: D, Diode_THT:D_A-405_P7.62mm_Horizontal, B.Cu at (137.2, 181.0)
- added D_C5: D, Diode_THT:D_A-405_P7.62mm_Horizontal, B.Cu at (156.2, 181.0)
- added D_C6: D, Diode_THT:D_A-405_P7.62mm_Horizontal, B.Cu at (175.3, 181.0)
- added D_C7: D, Diode_THT:D_A-405_P7.62mm_Horizontal, B.Cu at (200.7, 181.0)
- added D_C8: D, Diode_THT:D_A-405_P7.62mm_Horizontal, B.Cu at (219.7, 181.0)
- added D_C9: D, Diode_THT:D_A-405_P7.62mm_Horizontal, B.Cu at (238.8, 181.0)
- added D_D1: D, Diode_THT:D_A-405_P7.62mm_Horizontal, B.Cu at (80.0, 161.9)
- added D_D10: D, Diode_THT:D_A-405_P7.62mm_Horizontal, B.Cu at (254.0, 161.9)
- added D_D11: D, Diode_THT:D_A-405_P7.62mm_Horizontal, B.Cu at (283.2, 161.9)
- added D_D12: D, Diode_THT:D_A-405_P7.62mm_Horizontal, B.Cu at (302.3, 161.9)
- added D_D13: D, Diode_THT:D_A-405_P7.62mm_Horizontal, B.Cu at (321.3, 161.9)
- added D_D14: D, Diode_THT:D_A-405_P7.62mm_Horizontal, B.Cu at (340.4, 161.9)
- added D_D15: D, Diode_THT:D_A-405_P7.62mm_Horizontal, B.Cu at (359.4, 161.9)
- added D_D16: D, Diode_THT:D_A-405_P7.62mm_Horizontal, B.Cu at (378.5, 161.9)
- added D_D2: D, Diode_THT:D_A-405_P7.62mm_Horizontal, B.Cu at (99.1, 161.9)
- added D_D3: D, Diode_THT:D_A-405_P7.62mm_Horizontal, B.Cu at (118.1, 161.9)
- added D_D4: D, Diode_THT:D_A-405_P7.62mm_Horizontal, B.Cu at (137.2, 161.9)
- added D_D5: D, Diode_THT:D_A-405_P7.62mm_Horizontal, B.Cu at (156.2, 161.9)
- added D_D6: D, Diode_THT:D_A-405_P7.62mm_Horizontal, B.Cu at (175.3, 161.9)
- added D_D7: D, Diode_THT:D_A-405_P7.62mm_Horizontal, B.Cu at (200.7, 161.9)
- added D_D8: D, Diode_THT:D_A-405_P7.62mm_Horizontal, B.Cu at (219.7, 161.9)
- added D_D9: D, Diode_THT:D_A-405_P7.62mm_Horizontal, B.Cu at (238.8, 161.9)
- added D_E1: D, Diode_THT:D_A-405_P7.62mm_Horizontal, B.Cu at (80.0, 142.9)
- added D_E10: D, Diode_THT:D_A-405_P7.62mm_Horizontal, B.Cu at (257.8, 142.9)
- added D_E11: D, Diode_THT:D_A-405_P7.62mm_Horizontal, B.Cu at (283.2, 142.9)
- added D_E12: D, Diode_THT:D_A-405_P7.62mm_Horizontal, B.Cu at (302.3, 142.9)
- added D_E13: D, Diode_THT:D_A-405_P7.62mm_Horizontal, B.Cu at (321.3, 142.9)
- added D_E14: D, Diode_THT:D_A-405_P7.62mm_Horizontal, B.Cu at (340.4, 142.9)
- added D_E15: D, Diode_THT:D_A-405_P7.62mm_Horizontal, B.Cu at (359.4, 142.9)
- added D_E16: D, Diode_THT:D_A-405_P7.62mm_Horizontal, B.Cu at (378.5, 142.9)
- added D_E2: D, Diode_THT:D_A-405_P7.62mm_Horizontal, B.Cu at (99.1, 142.9)
- added D_E3: D, Diode_THT:D_A-405_P7.62mm_Horizontal, B.Cu at (118.1, 142.9)
- added D_E4: D, Diode_THT:D_A-405_P7.62mm_Horizontal, B.Cu at (137.2, 142.9)
- added D_E5: D, Diode_THT:D_A-405_P7.62mm_Horizontal, B.Cu at (156.2, 142.9)
- added D_E6: D, Diode_THT:D_A-405_P7.62mm_Horizontal, B.Cu at (175.3, 142.9)
- added D_E7: D, Diode_THT:D_A-405_P7.62mm_Horizontal, B.Cu at (200.7, 142.9)
- added D_E8: D, Diode_THT:D_A-405_P7.62mm_Horizontal, B.Cu at (219.7, 142.9)
- added D_E9: D, Diode_THT:D_A-405_P7.62mm_Horizontal, B.Cu at (238.8, 142.9)
- added J1: USB_B, custom:captive USB, F.Cu at (195.6, 130.8)
- added J2: Conn_01x05_Male, Connector_PinHeader_2.54mm:PinHeader_1x05_P2.54mm_Horizontal, B.Cu at (186.7, 181.0)
- added R1: 1k, Resistor_THT:R_Axial_DIN0207_L6.3mm_D2.5mm_P10.16mm_Horizontal, B.Cu at (93.3, 137.8)
- added R2: 1k, Resistor_THT:R_Axial_DIN0207_L6.3mm_D2.5mm_P10.16mm_Horizontal, B.Cu at (131.4, 137.8)
- added R3: 1k, Resistor_THT:R_Axial_DIN0207_L6.3mm_D2.5mm_P10.16mm_Horizontal, B.Cu at (169.5, 137.8)
- added R4: 1k, Resistor_THT:R_Axial_DIN0207_L6.3mm_D2.5mm_P10.16mm_Horizontal, B.Cu at (214.0, 137.8)
- added R5: 1k, Resistor_THT:R_Axial_DIN0207_L6.3mm_D2.5mm_P10.16mm_Horizontal, B.Cu at (252.1, 137.8)
- added R6: 1k, Resistor_THT:R_Axial_DIN0207_L6.3mm_D2.5mm_P10.16mm_Horizontal, B.Cu at (296.5, 137.8)
- added R7: 1k, Resistor_THT:R_Axial_DIN0207_L6.3mm_D2.5mm_P10.16mm_Horizontal, B.Cu at (334.6, 137.8)
- added R8: 1k, Resistor_THT:R_Axial_DIN0207_L6.3mm_D2.5mm_P10.16mm_Horizontal, B.Cu at (372.7, 137.8)
- added R9: 10k, Resistor_THT:R_Axial_DIN0207_L6.3mm_D2.5mm_P10.16mm_Horizontal, B.Cu at (188.0, 125.7)
- added REF**: cable tie, custom:cable tie, F.Cu at (202.6, 123.2)
- added REF**: MountingHole_3.2mm_M3, MountingHole:MountingHole_3.2mm_M3, F.Cu at (191.8, 119.4)
- added REF**: cable tie, custom:cable tie, F.Cu at (212.1, 123.2)
- added REF**: MountingHole_3.2mm_M3, MountingHole:MountingHole_3.2mm_M3, F.Cu at (396.2, 119.4)
- added REF**: MountingHole_3.2mm_M3, MountingHole:MountingHole_3.2mm_M3, F.Cu at (396.2, 223.5)
- added REF**: MountingHole_3.2mm_M3, MountingHole:MountingHole_3.2mm_M3, F.Cu at (69.8, 223.5)
- added REF**: MountingHole_3.2mm_M3, MountingHole:MountingHole_3.2mm_M3, F.Cu at (69.8, 119.4)
- added REF**: MountingHole_3.2mm_M3, MountingHole:MountingHole_3.2mm_M3, F.Cu at (191.8, 223.5)
- added REF**: MountingHole_3.2mm_M3, MountingHole:MountingHole_3.2mm_M3, F.Cu at (274.3, 223.5)
- added REF**: MountingHole_3.2mm_M3, MountingHole:MountingHole_3.2mm_M3, F.Cu at (274.3, 119.4)
- added SW1: SW_Push, custom:TE FSM4JAH, B.Cu at (191.8, 175.3)
- added SW_A1: SW_Push, custom:SW_Cherry_MX1A_1.00u_Plate_with_mounting_hole, F.Cu at (83.8, 209.6)
- added SW_A10: SW_Push, custom:SW_Cherry_MX1A_1.00u_Plate_with_mounting_hole, F.Cu at (261.6, 209.6)
- added SW_A11: SW_Push, custom:SW_Cherry_MX1A_1.00u_Plate_with_mounting_hole, F.Cu at (287.0, 209.6)
- added SW_A12: SW_Push, custom:SW_Cherry_MX1A_1.00u_Plate_with_mounting_hole, F.Cu at (306.1, 209.6)
- added SW_A13: SW_Push, custom:SW_Cherry_MX1A_1.00u_Plate_with_mounting_hole, F.Cu at (325.1, 209.6)
- added SW_A14: SW_Push, custom:SW_Cherry_MX1A_1.00u_Plate_with_mounting_hole, F.Cu at (344.2, 209.6)
- added SW_A15: SW_Push, custom:SW_Cherry_MX1A_1.00u_Plate_with_mounting_hole, F.Cu at (363.2, 209.6)
- added SW_A16: SW_Push, custom:SW_Cherry_MX1A_1.00u_Plate_with_mounting_hole, F.Cu at (382.3, 209.6)
- added SW_A2: SW_Push, custom:SW_Cherry_MX1A_1.00u_Plate_with_mounting_hole, F.Cu at (102.9, 209.6)
- added SW_A3: SW_Push, custom:SW_Cherry_MX1A_1.00u_Plate_with_mounting_hole, F.Cu at (121.9, 209.6)
- added SW_A4: SW_Push, custom:SW_Cherry_MX1A_1.00u_Plate_with_mounting_hole, F.Cu at (141.0, 209.6)
- added SW_A5: SW_Push, custom:SW_Cherry_MX1A_1.00u_Plate_with_mounting_hole, F.Cu at (160.0, 209.6)
- added SW_A6: SWA6, custom:SW_Cherry_MX1A_1.00u_Plate_with_mounting_hole, F.Cu at (179.1, 209.6)
- added SW_A7: SW_Push, custom:SW_Cherry_MX1A_1.00u_Plate_with_mounting_hole, F.Cu at (204.5, 209.6)
- added SW_A8: SW_Push, custom:SW_Cherry_MX1A_1.00u_Plate_with_mounting_hole, F.Cu at (223.5, 209.6)
- added SW_A9: SW_Push, custom:SW_Cherry_MX1A_1.00u_Plate_with_mounting_hole, F.Cu at (242.6, 209.6)
- added SW_B1: SW_Push, custom:SW_Cherry_MX1A_1.00u_Plate_with_mounting_hole, F.Cu at (83.8, 190.5)
- added SW_B10: SW_Push, custom:SW_Cherry_MX1A_1.00u_Plate_with_mounting_hole, F.Cu at (261.6, 190.5)
- added SW_B11: SW_Push, custom:SW_Cherry_MX1A_1.00u_Plate_with_mounting_hole, F.Cu at (287.0, 190.5)
- added SW_B12: SW_Push, custom:SW_Cherry_MX1A_1.00u_Plate_with_mounting_hole, F.Cu at (306.1, 190.5)
- added SW_B13: SW_Push, custom:SW_Cherry_MX1A_1.00u_Plate_with_mounting_hole, F.Cu at (325.1, 190.5)
- added SW_B14: SW_Push, custom:SW_Cherry_MX1A_1.00u_Plate_with_mounting_hole, F.Cu at (344.2, 190.5)
- added SW_B15: SW_Push, custom:SW_Cherry_MX1A_1.00u_Plate_with_mounting_hole, F.Cu at (363.2, 190.5)
- added SW_B16: SW_Push, custom:SW_Cherry_MX1A_1.00u_Plate_with_mounting_hole, F.Cu at (382.3, 190.5)
- added SW_B2: SW_Push, custom:SW_Cherry_MX1A_1.00u_Plate_with_mounting_hole, F.Cu at (102.9, 190.5)
- added SW_B3: SW_Push, custom:SW_Cherry_MX1A_1.00u_Plate_with_mounting_hole, F.Cu at (121.9, 190.5)
- added SW_B4: SW_Push, custom:SW_Cherry_MX1A_1.00u_Plate_with_mounting_hole, F.Cu at (141.0, 190.5)
- added SW_B5: SW_Push, custom:SW_Cherry_MX1A_1.00u_Plate_with_mounting_hole, F.Cu at (160.0, 190.5)
- added SW_B6: SWA6, custom:SW_Cherry_MX1A_1.00u_Plate_with_mounting_hole, F.Cu at (179.1, 190.5)
- added SW_B7: SW_Push, custom:SW_Cherry_MX1A_1.00u_Plate_with_mounting_hole, F.Cu at (204.5, 190.5)
- added SW_B8: SW_Push, custom:SW_Cherry_MX1A_1.00u_Plate_with_mounting_hole, F.Cu at (223.5, 190.5)
- added SW_B9: SW_Push, custom:SW_Cherry_MX1A_1.00u_Plate_with_mounting_hole, F.Cu at (242.6, 190.5)
- added SW_C1: SW_Push, custom:SW_Cherry_MX1A_1.00u_Plate_with_mounting_hole, F.Cu at (83.8, 171.4)
- added SW_C10: SW_Push, custom:SW_Cherry_MX1A_1.00u_Plate_with_mounting_hole, F.Cu at (261.6, 171.4)
- added SW_C11: SW_Push, custom:SW_Cherry_MX1A_1.00u_Plate_with_mounting_hole, F.Cu at (287.0, 171.4)
- added SW_C12: SW_Push, custom:SW_Cherry_MX1A_1.00u_Plate_with_mounting_hole, F.Cu at (306.1, 171.4)
- added SW_C13: SW_Push, custom:SW_Cherry_MX1A_1.00u_Plate_with_mounting_hole, F.Cu at (325.1, 171.4)
- added SW_C14: SW_Push, custom:SW_Cherry_MX1A_1.00u_Plate_with_mounting_hole, F.Cu at (344.2, 171.4)
- added SW_C15: SW_Push, custom:SW_Cherry_MX1A_1.00u_Plate_with_mounting_hole, F.Cu at (363.2, 171.4)
- added SW_C16: SW_Push, custom:SW_Cherry_MX1A_1.00u_Plate_with_mounting_hole, F.Cu at (382.3, 171.4)
- added SW_C2: SW_Push, custom:SW_Cherry_MX1A_1.00u_Plate_with_mounting_hole, F.Cu at (102.9, 171.4)
- added SW_C3: SW_Push, custom:SW_Cherry_MX1A_1.00u_Plate_with_mounting_hole, F.Cu at (121.9, 171.4)
- added SW_C4: SW_Push, custom:SW_Cherry_MX1A_1.00u_Plate_with_mounting_hole, F.Cu at (141.0, 171.4)
- added SW_C5: SW_Push, custom:SW_Cherry_MX1A_1.00u_Plate_with_mounting_hole, F.Cu at (160.0, 171.4)
- added SW_C6: SWA6, custom:SW_Cherry_MX1A_1.00u_Plate_with_mounting_hole, F.Cu at (179.1, 171.4)
- added SW_C7: SW_Push, custom:SW_Cherry_MX1A_1.00u_Plate_with_mounting_hole, F.Cu at (204.5, 171.4)
- added SW_C8: SW_Push, custom:SW_Cherry_MX1A_1.00u_Plate_with_mounting_hole, F.Cu at (223.5, 171.4)
- added SW_C9: SW_Push, custom:SW_Cherry_MX1A_1.00u_Plate_with_mounting_hole, F.Cu at (242.6, 171.4)
- added SW_D1: SW_Push, custom:SW_Cherry_MX1A_1.00u_Plate_with_mounting_hole, F.Cu at (83.8, 152.4)
- added SW_D10: SW_Push, custom:SW_Cherry_MX1A_1.00u_Plate_with_mounting_hole, F.Cu at (261.6, 152.4)
- added SW_D11: SW_Push, custom:SW_Cherry_MX1A_1.00u_Plate_with_mounting_hole, F.Cu at (287.0, 152.4)
- added SW_D12: SW_Push, custom:SW_Cherry_MX1A_1.00u_Plate_with_mounting_hole, F.Cu at (306.1, 152.4)
- added SW_D13: SW_Push, custom:SW_Cherry_MX1A_1.00u_Plate_with_mounting_hole, F.Cu at (325.1, 152.4)
- added SW_D14: SW_Push, custom:SW_Cherry_MX1A_1.00u_Plate_with_mounting_hole, F.Cu at (344.2, 152.4)
- added SW_D15: SW_Push, custom:SW_Cherry_MX1A_1.00u_Plate_with_mounting_hole, F.Cu at (363.2, 152.4)
- added SW_D16: SW_Push, custom:SW_Cherry_MX1A_1.00u_Plate_with_mounting_hole, F.Cu at (382.3, 152.4)
- added SW_D2: SW_Push, custom:SW_Cherry_MX1A_1.00u_Plate_with_mounting_hole, F.Cu at (102.9, 152.4)
- added SW_D3: SW_Push, custom:SW_Cherry_MX1A_1.00u_Plate_with_mounting_hole, F.Cu at (121.9, 152.4)
- added SW_D4: SW_Push, custom:SW_Cherry_MX1A_1.00u_Plate_with_mounting_hole, F.Cu at (141.0, 152.4)
- added SW_D5: SW_Push, custom:SW_Cherry_MX1A_1.00u_Plate_with_mounting_hole, F.Cu at (160.0, 152.4)
- added SW_D6: SWA6, custom:SW_Cherry_MX1A_1.00u_Plate_with_mounting_hole, F.Cu at (179.1, 152.4)
- added SW_D7: SW_Push, custom:SW_Cherry_MX1A_1.00u_Plate_with_mounting_hole, F.Cu at (204.5, 152.4)
- added SW_D8: SW_Push, custom:SW_Cherry_MX1A_1.00u_Plate_with_mounting_hole, F.Cu at (223.5, 152.4)
- added SW_D9: SW_Push, custom:SW_Cherry_MX1A_1.00u_Plate_with_mounting_hole, F.Cu at (242.6, 152.4)
- added SW_E1: SW_Push, custom:SW_Cherry_MX1A_1.00u_Plate_with_mounting_hole, F.Cu at (83.8, 133.3)
- added SW_E10: SW_Push, custom:SW_Cherry_MX1A_1.00u_Plate_with_mounting_hole, F.Cu at (261.6, 133.3)
- added SW_E11: SW_Push, custom:SW_Cherry_MX1A_1.00u_Plate_with_mounting_hole, F.Cu at (287.0, 133.3)
- added SW_E12: SW_Push, custom:SW_Cherry_MX1A_1.00u_Plate_with_mounting_hole, F.Cu at (306.1, 133.3)
- added SW_E13: SW_Push, custom:SW_Cherry_MX1A_1.00u_Plate_with_mounting_hole, F.Cu at (325.1, 133.3)
- added SW_E14: SW_Push, custom:SW_Cherry_MX1A_1.00u_Plate_with_mounting_hole, F.Cu at (344.2, 133.3)
- added SW_E15: SW_Push, custom:SW_Cherry_MX1A_1.00u_Plate_with_mounting_hole, F.Cu at (363.2, 133.3)
- added SW_E16: SW_Push, custom:SW_Cherry_MX1A_1.00u_Plate_with_mounting_hole, F.Cu at (382.3, 133.3)
- added SW_E2: SW_Push, custom:SW_Cherry_MX1A_1.00u_Plate_with_mounting_hole, F.Cu at (102.9, 133.3)
- added SW_E3: SW_Push, custom:SW_Cherry_MX1A_1.00u_Plate_with_mounting_hole, F.Cu at (121.9, 133.3)
- added SW_E4: SW_Push, custom:SW_Cherry_MX1A_1.00u_Plate_with_mounting_hole, F.Cu at (141.0, 133.3)
- added SW_E5: SW_Push, custom:SW_Cherry_MX1A_1.00u_Plate_with_mounting_hole, F.Cu at (160.0, 133.3)
- added SW_E6: SWA6, custom:SW_Cherry_MX1A_1.00u_Plate_with_mounting_hole, F.Cu at (179.1, 133.3)
- added SW_E7: SW_Push, custom:SW_Cherry_MX1A_1.00u_Plate_with_mounting_hole, F.Cu at (204.5, 133.3)
- added SW_E8: SW_Push, custom:SW_Cherry_MX1A_1.00u_Plate_with_mounting_hole, F.Cu at (223.5, 133.3)
- added SW_E9: SW_Push, custom:SW_Cherry_MX1A_1.00u_Plate_with_mounting_hole, F.Cu at (242.6, 133.3)
- added TP1: TestPoint, custom:test point 1mm, B.Cu at (194.9, 163.8)
- added TP2: TestPoint, custom:test point 1mm, B.Cu at (191.8, 163.8)
- added TP3: TestPoint, custom:test point 1mm, B.Cu at (188.6, 163.8)
- added U1: PIC16F1454-IP, Package_DIP:DIP-14_W7.62mm_Socket, B.Cu at (195.6, 144.1)
- added U2: PIC16F18855-IP, Package_DIP:DIP-28_W7.62mm_Socket, B.Cu at (278.1, 141.6)
Other:
- board outline added: 339.1 x 116.8 mm

Commit message: Get design rules set up for JLCPCB
Also make silkscreen text slightly thicker.
Other:
- net class Default: clearance 0.1524 -> 0.127; trace_width 0.1524 -> 0.127; via_dia 0.452 -> 0.6
- rule trace_clearance: 0.1524 -> 0.127
- rule trace_min: 0.1524 -> 0.127
- rule via_min_size: 0.452 -> 0.6

Commit message: checkpoint reached
Parts:
- J1: value USB_B -> USB_B_no_shield
- moved REF** 3.70 mm to (199.4, 121.3)
- moved REF** 3.70 mm to (208.9, 121.3)
- moved J1 2.84 mm to (193.0, 132.1)
Connections:
- U1 pad 2: Net-(U1-Pad2) -> GND
- U2 pad 23: Net-(U2-Pad23) -> GND
- U2 pad 24: Net-(U2-Pad24) -> GND
Routing:
- net /ROW5: track 0.00 -> 325.7 mm
- net /ROW1: track 0.00 -> 325.0 mm
- net /ROW3: track 0.00 -> 324.6 mm
- net /ROW9: track 0.00 -> 323.9 mm
- net /ROW7: track 0.00 -> 323.0 mm
- net /ROW4: track 0.00 -> 300.2 mm
- net /ROW6: track 0.00 -> 291.8 mm
- net /ROW8: track 0.00 -> 287.5 mm
- net /ROW10: track 0.00 -> 287.1 mm
- net /ROW2: track 0.00 -> 286.9 mm
- net /COL6: track 0.00 -> 203.4 mm
- net /COL5: track 0.00 -> 200.7 mm
- net /COL4: track 0.00 -> 199.7 mm
- net /COL8: track 0.00 -> 199.7 mm
- net /COL7: track 0.00 -> 199.7 mm
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- added copper zone on B.Cu, net GND

Commit message: Almost done routing!
Routing:
- net /COL1: track 199.7 -> 451.6 mm, vias 0 -> 2
- net /COL2: track 199.7 -> 412.0 mm, vias 0 -> 2
- net /COL3: track 199.7 -> 372.3 mm, vias 0 -> 2
- net VDD: track 26.3 -> 180.4 mm
- net /COL8: track 199.7 -> 339.1 mm, vias 0 -> 2
- net /COL4: track 199.7 -> 326.4 mm, vias 0 -> 2
- net /COL7: track 199.7 -> 298.2 mm, vias 0 -> 2
- net /~MCLR~_INT: track 0.00 -> 93.9 mm
- net /COL5: track 200.7 -> 287.7 mm, vias 0 -> 2
- net /~MCLR~_EXT: track 6.50 -> 67.4 mm, vias 0 -> 1
- net /ROW1: track 325.0 -> 368.6 mm, vias 0 -> 1
- net /ROW2: track 286.9 -> 325.1 mm, vias 0 -> 1
- net /ICSPCLK_EXT: track 0.00 -> 36.8 mm
- net /ICSPDAT_EXT: track 0.00 -> 36.3 mm
- net /ROW10: track 287.1 -> 314.5 mm, vias 0 -> 1
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
Commit message: ground planes ground plANES GROUND PLANES GR
Routing:
- net GND: track 13.3 -> 2.54 mm, vias 4 -> 3
- net /ICSPCLK_INT: track 99.7 -> 103.1 mm
- net VDD: track 180.4 -> 179.2 mm
- added copper zone on F.Cu, net GND

Commit message: Space holes a bit further out (I think)
Parts:
- moved REF** 4.84 mm to (203.8, 119.4)
- moved REF** 4.84 mm to (213.4, 119.4)
- moved REF** 0.90 mm to (396.9, 118.7)
- moved REF** 0.90 mm to (396.9, 224.2)
- moved REF** 0.90 mm to (69.2, 224.2)
- moved REF** 0.90 mm to (69.2, 118.7)
- moved REF** 0.63 mm to (191.8, 118.7)
- moved REF** 0.63 mm to (191.8, 224.2)
- moved REF** 0.63 mm to (274.3, 224.2)
- moved REF** 0.63 mm to (274.3, 118.7)
Routing:
- net GND: vias 3 -> 4

Commit message: Add some cut lines for laser cutting
Parts:
- REF** (x8): value MountingHole_3.2mm_M3 -> M3_hole; footprint MountingHole:MountingHole_3.2mm_M3 -> custom:M3_hole
- moved D_A13 34.7 mm to (307.3, 187.3)
- moved D_A14 34.7 mm to (326.4, 187.3)
- moved D_A15 34.7 mm to (345.4, 187.3)
- moved D_B13 34.7 mm to (307.3, 168.3)
- moved D_B14 34.7 mm to (326.4, 168.3)
- moved D_B15 34.7 mm to (345.4, 168.3)
- moved D_C13 34.7 mm to (307.3, 149.2)
- moved D_C14 34.7 mm to (326.4, 149.2)
- moved D_C15 34.7 mm to (345.4, 149.2)
- moved D_D13 34.7 mm to (307.3, 130.2)
- moved D_D14 34.7 mm to (326.4, 130.2)
- moved D_D15 34.7 mm to (345.4, 130.2)
- moved D_E13 34.7 mm to (307.3, 111.1)
- moved D_E14 34.7 mm to (326.4, 111.1)
- moved D_E15 34.7 mm to (345.4, 111.1)
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Other:
- outline, holes or cut-outs redrawn
- rule pad_to_mask_clearance: 0.0508 -> 0.2
