File: hardware/keyboard2018.kicad_pcb (KiCad board)
At the start: 2 copper layers, 342.9 x 120.7 mm, 190 parts, among them J1 USB_B_no_shield, J2 Conn_01x05_Male, SW1 SW_Push, U1 PIC16F1454-IP, U2 PIC16F18855-IP

Commit message: *Now* we're done
Other:
- rule pad_to_mask_clearance: 0.2 -> 0.0508
- board text added: "MKF"
- board text removed: "kbie MKF"
Changed lines of the file:
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@@
   (general
     (thickness 1.6)
-    (drawings 74)
+    (drawings 83)
     (tracks 1076)
     (zones 0)
@@
     (38 B.Mask user)
     (39 F.Mask user)
-    (40 Dwgs.User user hide)
+    (40 Dwgs.User user)
     (41 Cmts.User user)
     (42 Eco1.User user)
-    (43 Eco2.User user)
-    (44 Edge.Cuts user)
+    (43 Eco2.User user hide)
+    (44 Edge.Cuts user hide)
     (45 Margin user hide)
     (46 B.CrtYd user hide)
@@
     (pad_size 1.524 1.524)
     (pad_drill 0.762)
-    (pad_to_mask_clearance 0.2)
+    (pad_to_mask_clearance 0.0508)
     (aux_axis_origin 0 0)
     (visible_elements FFFFFF7F)
@@
   (module "custom:captive USB" (layer F.Cu)
     (at 181.61 100.33 270)
-    (fp_text reference J1 (at -6.35 0 270) (layer B.SilkS)
+    (fp_text reference J1 (at 0 1.905 270) (layer B.SilkS)
       (effects (font (size 1 1) (thickness 0.2032)) (justify mirror))
     )
@@
     (descr "Through hole angled pin header, 1x05, 2.54mm pitch, 6mm pin length, single row")
     (tags "Through hole angled pin header THT 1x05 2.54mm single row")
-    (fp_text reference J2 (at 0 -13.335 270) (layer B.SilkS)
+    (fp_text reference J2 (at -2.54 0) (layer B.SilkS)
       (effects (font (size 1 1) (thickness 0.2032)) (justify mirror))
     )
@@
   (module "custom:TE FSM4JAH" (layer B.Cu)
     (at 177.875 143.565 180)
-    (fp_text reference SW1 (at 0 6.985 180) (layer B.SilkS)
+    (fp_text reference SW1 (at 0.075 2.595 180) (layer B.SilkS)
       (effects (font (size 1 1) (thickness 0.2032)) (justify mirror))
     )
@@
     )
   )
+  (gr_text MKF (at 260.35 177.8) (layer B.SilkS)
+    (effects (font (size 2.54 2.54) (thickness 0.4064)) (justify mirror))
+  )
+  (gr_line (start 184.15 147.32) (end 182.88 147.32) (layer B.SilkS) (width 0.2032))
+  (gr_line (start 182.88 146.05) (end 184.15 147.32) (layer B.SilkS) (width 0.2032))
+  (gr_line (start 181.61 147.32) (end 182.88 146.05) (layer B.SilkS) (width 0.2032))
+  (gr_line (start 182.88 147.32) (end 181.61 147.32) (layer B.SilkS) (width 0.2032))
+  (gr_line (start 182.88 147.955) (end 182.88 147.32) (layer B.SilkS) (width 0.2032))
+  (gr_line (start 268.605 90.17) (end 372.11 90.17) (layer Eco1.User) (width 0.0508))
+  (gr_line (start 252.095 189.23) (end 186.055 189.23) (layer Eco1.User) (width 0.0508))
+  (gr_line (start 169.545 189.23) (end 66.04 189.23) (layer Eco1.User) (width 0.0508))
   (gr_text kbie (at 69.85 84.455) (layer F.SilkS)
     (effects (font (size 2.54 2.54) (thickness 0.4064)))
@@
   )
   (gr_circle (center 177.8 141.605) (end 193.04 141.605) (layer Eco1.User) (width 0.0508))
-  (gr_text "kbie\nMKF" (at 177.8 168.275) (layer B.SilkS)
+  (gr_text kbie (at 260.35 158.75) (layer B.SilkS)
     (effects (font (size 2.54 2.54) (thickness 0.4064)) (justify mirror))
   )
   (gr_line (start 186.055 79.248) (end 203.2 79.248) (layer Eco1.User) (width 0.0508))
   (gr_line (start 203.2 79.248) (end 382.905 79.248) (layer Eco1.User) (width 0.0508))
-  (gr_line (start 203.2 90.17) (end 372.11 90.17) (layer Eco1.User) (width 0.0508))
+  (gr_line (start 203.2 90.17) (end 252.095 90.17) (layer Eco1.User) (width 0.0508))
   (gr_line (start 186.055 90.17) (end 203.2 90.17) (layer Eco1.User) (width 0.0508))
   (gr_arc (start 203.2 81.153) (end 203.2 79.248) (angle -90) (layer Eco1.User) (width 0.0508))
@@
   (gr_arc (start 382.905 86.995) (end 390.525 86.995) (angle -90) (layer Edge.Cuts) (width 0.0508))
   (gr_line (start 58.42 181.61) (end 58.42 97.79) (layer Eco1.User) (width 0.0508))
-  (gr_line (start 372.11 189.23) (end 66.04 189.23) (layer Eco1.User) (width 0.0508))
+  (gr_line (start 372.11 189.23) (end 268.605 189.23) (layer Eco1.User) (width 0.0508))
   (gr_line (start 379.73 97.79) (end 379.73 181.61) (layer Eco1.User) (width 0.0508))
   (gr_line (start 66.04 90.17) (end 169.545 90.17) (layer Eco1.User) (width 0.0508))
@@
     (polygon
       (pts
-        (xy 59.69 186.69) (xy 59.69 93.98) (xy 62.23 91.44) (xy 173.99 91.44) (xy 175.26 92.71)
-        (xy 180.34 92.71) (xy 181.61 91.44) (xy 256.54 91.44) (xy 257.81 92.71) (xy 262.89 92.71)
-        (xy 264.16 91.44) (xy 375.92 91.44) (xy 378.46 93.98) (xy 378.46 186.69) (xy 375.92 189.23)
-        (xy 265.43 189.23) (xy 262.89 186.69) (xy 257.81 186.69) (xy 255.27 189.23) (xy 182.88 189.23)
-        (xy 180.34 186.69) (xy 175.26 186.69) (xy 172.72 189.23) (xy 62.23 189.23)
+        (xy 59.69 186.69) (xy 59.69 93.98) (xy 62.23 91.44) (xy 375.92 91.44) (xy 378.46 93.98)
+        (xy 378.46 186.69) (xy 375.92 189.23) (xy 62.23 189.23)
       )
     )

Commit message: Add some helpful text
Other:
- board text added: "3mm transparent cast acrylic"
- board text added: "4.5mm transparent cast acrylic"
- board text added: "6mm transparent cast acrylic"
Changed lines of the file:
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@@
   (general
     (thickness 1.6)
-    (drawings 83)
+    (drawings 87)
     (tracks 1076)
     (zones 0)
@@
     (41 Cmts.User user)
     (42 Eco1.User user)
-    (43 Eco2.User user hide)
+    (43 Eco2.User user)
     (44 Edge.Cuts user hide)
     (45 Margin user hide)
@@
     )
   )
+  (gr_text "3mm transparent cast acrylic" (at 311.785 229.87) (layer Cmts.User)
+    (effects (font (size 1.5 1.5) (thickness 0.3)) (justify left))
+  )
+  (gr_text "4.5mm transparent cast acrylic" (at 311.785 227.33) (layer Cmts.User)
+    (effects (font (size 1.5 1.5) (thickness 0.3)) (justify left))
+  )
+  (gr_text "6mm transparent cast acrylic" (at 311.785 224.79) (layer Cmts.User)
+    (effects (font (size 1.5 1.5) (thickness 0.3)) (justify left))
+  )
+  (gr_text "3mm transparent cast acrylic" (at 311.785 222.25) (layer Cmts.User)
+    (effects (font (size 1.5 1.5) (thickness 0.3)) (justify left))
+  )
   (gr_text MKF (at 260.35 177.8) (layer B.SilkS)
