File: hardware/matrix.sch (KiCad schematic (older format))
At the start: 168 parts

Commit message: Finish schematic again
Parts:
- SW_A1, SW_A10, SW_A11, SW_A12, SW_A13, SW_A14, SW_A15, SW_A16, SW_A2, SW_A3, SW_A4, SW_A5, SW_A6, SW_A7, SW_A8, SW_A9, SW_B1, SW_B10, SW_B11, SW_B12, SW_B13, SW_B14, SW_B15, SW_B16, SW_B2, SW_B3, SW_B4, SW_B5, SW_B6, SW_B7, SW_B8, SW_B9, SW_C1, SW_C10, SW_C11, SW_C12, SW_C13, SW_C14, SW_C15, SW_C16, SW_C2, SW_C3, SW_C4, SW_C5, SW_C6, SW_C7, SW_C8, SW_C9, SW_D1, SW_D10, SW_D11, SW_D12, SW_D13, SW_D14, SW_D15, SW_D16, SW_D2, SW_D3, SW_D4, SW_D5, SW_D6, SW_D7, SW_D8, SW_D9, SW_E1, SW_E10, SW_E11, SW_E12, SW_E13, SW_E14, SW_E15, SW_E16, SW_E2, SW_E3, SW_E4, SW_E5, SW_E6, SW_E7, SW_E8, SW_E9: footprint custom-switch:SW_Cherry_MX1A_1.00u_Plate_with_mounting_hole -> custom:SW_Cherry_MX1A_1.00u_Plate_with_mounting_hole

Commit message: I think it's done!
Parts:
- SW_A6, SW_B6, SW_C6, SW_D6, SW_E6: value SWA6 -> SW_Push
Changed lines of the file:
@@
 P 4850 4750
 F 0 "SW_A6" V 4850 4702 50  0000 R CNN
-F 1 "SWA6" V 4805 4702 50  0001 R CNN
+F 1 "SW_Push" V 4805 4702 50  0001 R CNN
 F 2 "custom:SW_Cherry_MX1A_1.00u_Plate_with_mounting_hole" H 4850 4950 50  0001 C CNN
 F 3 "" H 4850 4950 50  0001 C CNN
@@
 P 4850 3950
 F 0 "SW_B6" V 4850 3902 50  0000 R CNN
-F 1 "SWA6" V 4805 3902 50  0001 R CNN
+F 1 "SW_Push" V 4805 3902 50  0001 R CNN
 F 2 "custom:SW_Cherry_MX1A_1.00u_Plate_with_mounting_hole" H 4850 4150 50  0001 C CNN
 F 3 "" H 4850 4150 50  0001 C CNN
@@
 P 4850 3150
 F 0 "SW_C6" V 4850 3102 50  0000 R CNN
-F 1 "SWA6" V 4805 3102 50  0001 R CNN
+F 1 "SW_Push" V 4805 3102 50  0001 R CNN
 F 2 "custom:SW_Cherry_MX1A_1.00u_Plate_with_mounting_hole" H 4850 3350 50  0001 C CNN
 F 3 "" H 4850 3350 50  0001 C CNN
@@
 P 4850 2350
 F 0 "SW_D6" V 4850 2302 50  0000 R CNN
-F 1 "SWA6" V 4805 2302 50  0001 R CNN
+F 1 "SW_Push" V 4805 2302 50  0001 R CNN
 F 2 "custom:SW_Cherry_MX1A_1.00u_Plate_with_mounting_hole" H 4850 2550 50  0001 C CNN
 F 3 "" H 4850 2550 50  0001 C CNN
@@
 P 4850 1550
 F 0 "SW_E6" V 4850 1502 50  0000 R CNN
-F 1 "SWA6" V 4805 1502 50  0001 R CNN
+F 1 "SW_Push" V 4805 1502 50  0001 R CNN
 F 2 "custom:SW_Cherry_MX1A_1.00u_Plate_with_mounting_hole" H 4850 1750 50  0001 C CNN
 F 3 "" H 4850 1750 50  0001 C CNN
